File: csi.kicad_sch (KiCad schematic)
At the start: 65 parts, among them J7 Conn_FFC_WE_68715014522, J8 Conn_FFC_WE_68715014522, U24 AP22615A_TSOT26, U25 AP22615A_TSOT26, U26 PI4MSD5V9548AZDEX, U27 AP22615A_TSOT26, U28 AP22615A_TSOT26, U31 NTS0102_XSON, U32 NTS0102_XSON

Commit message: Adding libs/3d-models back from commit 51986f3981aa7fd18fc8cc0c4764f958b589b418
Parts:
- C100, C101, C42, C43, C89, C90, C91, C96, C97: value C_100n_0402 -> GRM155R61H104KE14D; MPN GRM155R61H104KE14D -> (none); Manufacturer Murata -> (none); Manufacturer 1 (none) -> Murata; Manufacturer Part Number 1 (none) -> GRM155R61H104KE14D; OldValue (none) -> C_100n_0402
- C94, C95, C98, C99: value C_1u_0402 -> C1005X6S1A105K050BC; MPN C1005X6S1A105K050BC -> (none); Manufacturer TDK -> (none); Manufacturer 1 (none) -> TDK; Manufacturer Part Number 1 (none) -> C1005X6S1A105K050BC; OldValue (none) -> C_1u_0402
- D18, D20, D24, D25: value LED_G_0603_LTST-C190GKT -> LTST-C190GKT; MPN LTST-C190GKT -> (none); Manufacturer Lite-On -> (none); Manufacturer 1 (none) -> Lite-On; Manufacturer Part Number 1 (none) -> LTST-C190GKT; OldValue (none) -> LED_G_0603_LTST-C190GKT
- J7, J8: value Conn_FFC_WE_68715014522 -> 68715014522; MPN 68715014522 -> (none); Manufacturer Würth Elektronik -> (none); Manufacturer 1 (none) -> Würth Elektronik; Manufacturer Part Number 1 (none) -> 68715014522; OldValue (none) -> Conn_FFC_WE_68715014522
- R10, R7, R8, R9: value R_4k7_0402 -> CR0402-FX-4701GLF; MPN CR0402-FX-4701GLF -> (none); Manufacturer Bourns -> (none); Manufacturer 1 (none) -> Bourns; Manufacturer Part Number 1 (none) -> CR0402-FX-4701GLF; OldValue (none) -> R_4k7_0402
- R103, R107, R108, R122, R50, R51: value R_4x0R_0201_array -> EXB-18VR000X; MPN EXB-18VR000X -> (none); Manufacturer Panasonic -> (none); Manufacturer 1 (none) -> Panasonic; Manufacturer Part Number 1 (none) -> EXB-18VR000X; OldValue (none) -> R_4x0R_0201_array
- R132, R133: value R_200R_0402 -> CR0402-FX-2000GLF; MPN CR0402-FX-2000GLF -> (none); Manufacturer Bourns -> (none); Manufacturer 1 (none) -> Bourns; Manufacturer Part Number 1 (none) -> CR0402-FX-2000GLF; OldValue (none) -> R_200R_0402
- R161, R162, R166, R167, R168, R171, R174, R179: value R_0R_0402 -> ERJ2GE0R00X; MPN ERJ2GE0R00X -> (none); Manufacturer Panasonic -> (none); Manufacturer 1 (none) -> Panasonic; Manufacturer Part Number 1 (none) -> ERJ2GE0R00X; OldValue (none) -> R_0R_0402
- R163, R193, R194, R66, R67: value R_10k_0402 -> CR0402-FX-1002GLF; MPN CR0402-FX-1002GLF -> (none); Manufacturer Bourns -> (none); Manufacturer 1 (none) -> Bourns; Manufacturer Part Number 1 (none) -> CR0402-FX-1002GLF; OldValue (none) -> R_10k_0402
- R180, R6: value R_100k_0402 -> CR0402-FX-1003GLF; MPN CR0402-FX-1003GLF -> (none); Manufacturer Bourns -> (none); Manufacturer 1 (none) -> Bourns; Manufacturer Part Number 1 (none) -> CR0402-FX-1003GLF; OldValue (none) -> R_100k_0402
- R197, R206: value R_470R_0402 -> CR0402-FX-4700GLF; MPN CR0402-FX-4700GLF -> (none); Manufacturer Bourns -> (none); Manufacturer 1 (none) -> Bourns; Manufacturer Part Number 1 (none) -> CR0402-FX-4700GLF; OldValue (none) -> R_470R_0402
- R36, R48: value R_4x2k2_0201_array -> EXB-18V222JX; MPN EXB-18V222JX -> (none); Manufacturer Panasonic -> (none); Manufacturer 1 (none) -> Panasonic; Manufacturer Part Number 1 (none) -> EXB-18V222JX; OldValue (none) -> R_4x2k2_0201_array
- TP36, TP37, TP38, TP39, TP40, TP41, TP42, TP43: OldValue (none) -> TP_0.75mm_SMD
- U24, U25, U27, U28: value AP22615A_TSOT26 -> AP22615AWU-7; MPN AP22615AWU-7 -> (none); Manufacturer Diodes Incorporated -> (none); Manufacturer 1 (none) -> Diodes Incorporated; Manufacturer Part Number 1 (none) -> AP22615AWU-7; OldValue (none) -> AP22615A_TSOT26
- U26: MPN PI4MSD5V9548AZDEX -> (none); Manufacturer Diodes Incorporated -> (none); Manufacturer 1 (none) -> Diodes Incorporated; Manufacturer Part Number 1 (none) -> PI4MSD5V9548AZDEX; OldValue (none) -> PI4MSD5V9548AZDEX
- U31, U32: value NTS0102_XSON -> NTS0102GT; MPN NTS0102GT -> (none); Manufacturer NXP -> (none); Manufacturer 1 (none) -> NXP; Manufacturer Part Number 1 (none) -> NTS0102GT; OldValue (none) -> NTS0102_XSON
