File: ethernet.kicad_sch (KiCad schematic)
At the start: 44 parts, among them J6 Bus_RJ45_5-2337992-8, Q17 PJE138K, U22 TPS2372-3RGWR, U23 ULS-12_5-D48N-C, U39 ACPL-217-500E

Commit message: Adding libs/3d-models back from commit 51986f3981aa7fd18fc8cc0c4764f958b589b418
Parts:
- C52, C78: value C_100n_0402 -> GRM155R61H104KE14D; MPN GRM155R61H104KE14D -> (none); Manufacturer Murata -> (none); Manufacturer 1 (none) -> Murata; Manufacturer Part Number 1 (none) -> GRM155R61H104KE14D; OldValue (none) -> C_100n_0402
- C76: value C_100n_100V_0805 -> CL21B104KCFNNNE; MPN CL21B104KCFNNNE -> (none); Manufacturer Samsung Electro-Mechanics -> (none); Manufacturer 1 (none) -> Samsung Electro-Mechanics; Manufacturer Part Number 1 (none) -> CL21B104KCFNNNE; OldValue (none) -> C_100n_100V_0805
- C77: value C_10n_0603 -> 06031C103JAT2A; MPN 06031C103JAT2A -> (none); Manufacturer AVX -> (none); Manufacturer 1 (none) -> AVX; Manufacturer Part Number 1 (none) -> 06031C103JAT2A; OldValue (none) -> C_10n_0603
- C79, C80, C81, C82: value C_22u_100V_2220 -> C5750X7S2A226M280KB; MPN C5750X7S2A226M280KB -> (none); Manufacturer TDK -> (none); Manufacturer 1 (none) -> TDK; Manufacturer Part Number 1 (none) -> C5750X7S2A226M280KB; OldValue (none) -> C_22u_100V_2220
- C84, C85: value C_47u_16V_1206 -> C3216X5R1C476M160AB; MPN C3216X5R1C476M160AB -> (none); Manufacturer TDK -> (none); Manufacturer 1 (none) -> TDK; Manufacturer Part Number 1 (none) -> C3216X5R1C476M160AB; OldValue (none) -> C_47u_16V_1206
- D12, D13: MPN CD-MMBL110S -> (none); Manufacturer Bourns -> (none); Manufacturer 1 (none) -> Bourns; Manufacturer Part Number 1 (none) -> CD-MMBL110S; OldValue (none) -> CD-MMBL110S
- D14: MPN PTVS58VS1UR,115 -> (none); Manufacturer Nexperia -> (none); Manufacturer 1 (none) -> Nexperia; Manufacturer Part Number 1 (none) -> PTVS58VS1UR,115; OldValue (none) -> PTVS58VS1UR,115
- D15: value LED_G_0603_LTST-C190GKT -> LTST-C190GKT; MPN LTST-C190GKT -> (none); Manufacturer Lite-On -> (none); Manufacturer 1 (none) -> Lite-On; Manufacturer Part Number 1 (none) -> LTST-C190GKT; OldValue (none) -> LED_G_0603_LTST-C190GKT
- FB2, FB3: value FB_220Z_2A_Murata-BLM21PG_0805 -> BLM21PG221SN1D; MPN BLM21PG221SN1D -> (none); Manufacturer Murata -> (none); Manufacturer 1 (none) -> Murata; Manufacturer Part Number 1 (none) -> BLM21PG221SN1D; OldValue (none) -> FB_220Z_2A_Murata-BLM21PG_0805
- J6: value Bus_RJ45_5-2337992-8 -> 5-2337992-8; MPN 5-2337992-8 -> (none); Manufacturer TE Connectivity -> (none); Manufacturer 1 (none) -> TE Connectivity; Manufacturer Part Number 1 (none) -> 5-2337992-8; OldValue (none) -> Bus_RJ45_5-2337992-8
- Q17: value PJE138K -> PJE138K_R1_00001; MPN PJE138K_R1_00001 -> (none); Manufacturer PANJIT -> (none); Manufacturer 1 (none) -> PANJIT; Manufacturer Part Number 1 (none) -> PJE138K_R1_00001; OldValue (none) -> PJE138K
- R123: value R_1k3_0402 -> CR0402-FX-1301GLF; MPN CR0402-FX-1301GLF -> (none); Manufacturer Bourns -> (none); Manufacturer 1 (none) -> Bourns; Manufacturer Part Number 1 (none) -> CR0402-FX-1301GLF; OldValue (none) -> R_1k3_0402
- R129, R241: value R_0R_0402 -> ERJ2GE0R00X; MPN ERJ2GE0R00X -> (none); Manufacturer Panasonic -> (none); Manufacturer 1 (none) -> Panasonic; Manufacturer Part Number 1 (none) -> ERJ2GE0R00X; OldValue (none) -> R_0R_0402
- R142: value R_49k9_0402 -> CR0402-FX-4992GLF; MPN CR0402-FX-4992GLF -> (none); Manufacturer Bourns -> (none); Manufacturer 1 (none) -> Bourns; Manufacturer Part Number 1 (none) -> CR0402-FX-4992GLF; OldValue (none) -> R_49k9_0402
- R145: value R_1k2_0402 -> CR0402-FX-1201GLF; MPN CR0402-FX-1201GLF -> (none); Manufacturer Bourns -> (none); Manufacturer 1 (none) -> Bourns; Manufacturer Part Number 1 (none) -> CR0402-FX-1201GLF; OldValue (none) -> R_1k2_0402
- R146, R154: value R_24k9_0402 -> CR0402-FX-2492GLF; MPN CR0402-FX-2492GLF -> (none); Manufacturer Bourns -> (none); Manufacturer 1 (none) -> Bourns; Manufacturer Part Number 1 (none) -> CR0402-FX-2492GLF; OldValue (none) -> R_24k9_0402
- R147, R151, R152: value R_200R_0402 -> CR0402-FX-2000GLF; MPN CR0402-FX-2000GLF -> (none); Manufacturer Bourns -> (none); Manufacturer 1 (none) -> Bourns; Manufacturer Part Number 1 (none) -> CR0402-FX-2000GLF; OldValue (none) -> R_200R_0402
- R148, R149, R150, R153: value R_10k_0402 -> CR0402-FX-1002GLF; MPN CR0402-FX-1002GLF -> (none); Manufacturer Bourns -> (none); Manufacturer 1 (none) -> Bourns; Manufacturer Part Number 1 (none) -> CR0402-FX-1002GLF; OldValue (none) -> R_10k_0402
- R155, R156: value R_1k_0402 -> CR0402-FX-1001GLF; MPN CR0402-FX-1001GLF -> (none); Manufacturer Bourns -> (none); Manufacturer 1 (none) -> Bourns; Manufacturer Part Number 1 (none) -> CR0402-FX-1001GLF; OldValue (none) -> R_1k_0402
- R157, R243: value R_0R_0603 -> CR0603-J/-000ELF; MPN CR0603-J/-000ELF -> (none); Manufacturer Bourns -> (none); Manufacturer 1 (none) -> Bourns; Manufacturer Part Number 1 (none) -> CR0603-J/-000ELF; OldValue (none) -> R_0R_0603
- R185, R229: value R_100k_0402 -> CR0402-FX-1003GLF; MPN CR0402-FX-1003GLF -> (none); Manufacturer Bourns -> (none); Manufacturer 1 (none) -> Bourns; Manufacturer Part Number 1 (none) -> CR0402-FX-1003GLF; OldValue (none) -> R_100k_0402
- R196: value R_63R4_0603 -> CR0603-FX-63R4ELF; MPN CR0603-FX-63R4ELF -> (none); Manufacturer Bourns -> (none); Manufacturer 1 (none) -> Bourns; Manufacturer Part Number 1 (none) -> CR0603-FX-63R4ELF; OldValue (none) -> R_63R4_0603
- R198, R199: value R_470k_0402 -> CR0402-FX-4703GLF; MPN CR0402-FX-4703GLF -> (none); Manufacturer Bourns -> (none); Manufacturer 1 (none) -> Bourns; Manufacturer Part Number 1 (none) -> CR0402-FX-4703GLF; OldValue (none) -> R_470k_0402
- U22: MPN TPS2372-3RGWR -> (none); Manufacturer Texas Instruments -> (none); Manufacturer 1 (none) -> Texas Instruments; Manufacturer Part Number 1 (none) -> TPS2372-3RGWR; OldValue (none) -> TPS2372-3RGWR
- U23: value ULS-12_5-D48N-C -> ULS-12/5-D48N-C; MPN ULS-12/5-D48N-C -> (none); Manufacturer Murata -> (none); Manufacturer 1 (none) -> Murata; Manufacturer Part Number 1 (none) -> ULS-12/5-D48N-C; OldValue (none) -> ULS-12_5-D48N-C
- U39: MPN ACPL-217-500E -> (none); Manufacturer Broadcom -> (none); Manufacturer 1 (none) -> Broadcom; Manufacturer Part Number 1 (none) -> ACPL-217-500E; OldValue (none) -> ACPL-217-500E
