File: hdmi.kicad_sch (KiCad schematic)
At the start: 58 parts, among them J13 HDMI-Mini-C_WE_685119136923, Q1 PJE138K, Q12 PJE138K, Q2 PJE138K, Q3 PJE138K, U36 TS3DV642RUARQ1, U43 NTS0102_XSON, U44 TPD4E05U06QDQARQ1, U45 TPD4E05U06QDQARQ1, U46 TPD4E05U06QDQARQ1

Commit message: Adding libs/3d-models back from commit 51986f3981aa7fd18fc8cc0c4764f958b589b418
Parts:
- C131, C132, C133, C135, C138, C139, C163, C164, C86, C87, C88, C92: value C_100n_0402 -> GRM155R61H104KE14D; MPN GRM155R61H104KE14D -> (none); Manufacturer Murata -> (none); Manufacturer 1 (none) -> Murata; Manufacturer Part Number 1 (none) -> GRM155R61H104KE14D; OldValue (none) -> C_100n_0402
- C47: value C_1u_0402 -> C1005X6S1A105K050BC; MPN C1005X6S1A105K050BC -> (none); Manufacturer TDK -> (none); Manufacturer 1 (none) -> TDK; Manufacturer Part Number 1 (none) -> C1005X6S1A105K050BC; OldValue (none) -> C_1u_0402
- C51: value C_10u_0603 -> GRM188R61A106KE69D; MPN GRM188R61A106KE69D -> (none); Manufacturer Murata -> (none); Manufacturer 1 (none) -> Murata; Manufacturer Part Number 1 (none) -> GRM188R61A106KE69D; OldValue (none) -> C_10u_0603
- D38: MPN RB521S30T1G -> (none); Manufacturer ON Semiconductor -> (none); Manufacturer 1 (none) -> ON Semiconductor; Manufacturer Part Number 1 (none) -> RB521S30T1G; OldValue (none) -> RB521S30T1G
- FB4: value FB_220Z_2A_Murata-BLM21PG_0805 -> BLM21PG221SN1D; MPN BLM21PG221SN1D -> (none); Manufacturer Murata -> (none); Manufacturer 1 (none) -> Murata; Manufacturer Part Number 1 (none) -> BLM21PG221SN1D; OldValue (none) -> FB_220Z_2A_Murata-BLM21PG_0805
- J13: value HDMI-Mini-C_WE_685119136923 -> 685119136923; MPN 685119136923 -> (none); Manufacturer Würth Elektronik -> (none); Manufacturer 1 (none) -> Würth Elektronik; Manufacturer Part Number 1 (none) -> 685119136923; OldValue (none) -> HDMI-Mini-C_WE_685119136923
- Q1, Q12, Q2, Q3: value PJE138K -> PJE138K_R1_00001; MPN PJE138K_R1_00001 -> (none); Manufacturer PANJIT -> (none); Manufacturer 1 (none) -> PANJIT; Manufacturer Part Number 1 (none) -> PJE138K_R1_00001; OldValue (none) -> PJE138K
- R160, R211, R228, R47, R49: value R_10k_0402 -> CR0402-FX-1002GLF; MPN CR0402-FX-1002GLF -> (none); Manufacturer Bourns -> (none); Manufacturer 1 (none) -> Bourns; Manufacturer Part Number 1 (none) -> CR0402-FX-1002GLF; OldValue (none) -> R_10k_0402
- R208, R227, R279, R280, R281, R282: value R_2k2_0402 -> CR0402-FX-2201GLF; MPN CR0402-FX-2201GLF -> (none); Manufacturer Bourns -> (none); Manufacturer 1 (none) -> Bourns; Manufacturer Part Number 1 (none) -> CR0402-FX-2201GLF; OldValue (none) -> R_2k2_0402
- R209, R210, R212, R213, R214, R220, R221, R224: value R_499R_0402 -> CR0402-FX-4990GLF; MPN CR0402-FX-4990GLF -> (none); Manufacturer Bourns -> (none); Manufacturer 1 (none) -> Bourns; Manufacturer Part Number 1 (none) -> CR0402-FX-4990GLF; OldValue (none) -> R_499R_0402
- R225, R226, R277, R278, R293, R40: value R_0R_0402 -> ERJ2GE0R00X; MPN ERJ2GE0R00X -> (none); Manufacturer Panasonic -> (none); Manufacturer 1 (none) -> Panasonic; Manufacturer Part Number 1 (none) -> ERJ2GE0R00X; OldValue (none) -> R_0R_0402
- R34, R35: value R_4x0R_0201_array -> EXB-18VR000X; MPN EXB-18VR000X -> (none); Manufacturer Panasonic -> (none); Manufacturer 1 (none) -> Panasonic; Manufacturer Part Number 1 (none) -> EXB-18VR000X; OldValue (none) -> R_4x0R_0201_array
- TP21, TP22, TP56, TP57, TP58: OldValue (none) -> TP_0.75mm_SMD
- U36: MPN TS3DV642RUARQ1 -> (none); Manufacturer Texas Instruments -> (none); Manufacturer 1 (none) -> Texas Instruments; Manufacturer Part Number 1 (none) -> TS3DV642RUARQ1; OldValue (none) -> TS3DV642RUARQ1
- U43: value NTS0102_XSON -> NTS0102GT; MPN NTS0102GT -> (none); Manufacturer NXP -> (none); Manufacturer 1 (none) -> NXP; Manufacturer Part Number 1 (none) -> NTS0102GT; OldValue (none) -> NTS0102_XSON
- U44, U45, U46: MPN TPD4E05U06QDQARQ1 -> (none); Manufacturer Texas Instruments -> (none); Manufacturer 1 (none) -> Texas Instruments; Manufacturer Part Number 1 (none) -> TPD4E05U06QDQARQ1; OldValue (none) -> TPD4E05U06QDQARQ1
