File: m-2.kicad_sch (KiCad schematic)
At the start: 61 parts, among them J1 Bus_M.2_2199230-6, J2 Bus_M.2_1-2199230-6, M3 Mech_M2_2280_H2.5mm, U2 74LVC2G07_SOT457, U3 74LVC2G07_SOT457, Y1 Oscillator_32.768kHz_ECS_2520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

Commit message: Adding libs/3d-models back from commit 51986f3981aa7fd18fc8cc0c4764f958b589b418
Parts:
- A2: OldValue (none) -> Mech_M2_2242_H2.5mm
- C10, C13, C14, C15, C16, C17, C18, C19, C20, C9: value C_220n_0402 -> CC0402KRX5R6BB224; MPN CC0402KRX5R6BB224 -> (none); Manufacturer YAGEO -> (none); Manufacturer 1 (none) -> YAGEO; Manufacturer Part Number 1 (none) -> CC0402KRX5R6BB224; OldValue (none) -> C_220n_0402
- C11, C12, C21, C22, C23, C24: value C_10u_0603 -> GRM188R61A106KE69D; MPN GRM188R61A106KE69D -> (none); Manufacturer Murata -> (none); Manufacturer 1 (none) -> Murata; Manufacturer Part Number 1 (none) -> GRM188R61A106KE69D; OldValue (none) -> C_10u_0603
- C25, C7, C8: value C_100n_0402 -> GRM155R61H104KE14D; MPN GRM155R61H104KE14D -> (none); Manufacturer Murata -> (none); Manufacturer 1 (none) -> Murata; Manufacturer Part Number 1 (none) -> GRM155R61H104KE14D; OldValue (none) -> C_100n_0402
- D1, D51, D52: value LED_G_0603_LTST-C190GKT -> LTST-C190GKT; MPN LTST-C190GKT -> (none); Manufacturer Lite-On -> (none); Manufacturer 1 (none) -> Lite-On; Manufacturer Part Number 1 (none) -> LTST-C190GKT; OldValue (none) -> LED_G_0603_LTST-C190GKT
- J1: value Bus_M.2_2199230-6 -> 2199230-6; MPN 2199230-6 -> (none); Manufacturer TE Connectivity -> (none); Manufacturer 1 (none) -> TE Connectivity; Manufacturer Part Number 1 (none) -> 2199230-6; OldValue (none) -> Bus_M.2_2199230-6
- J2: value Bus_M.2_1-2199230-6 -> 1-2199230-6; MPN 1-2199230-6 -> (none); Manufacturer TE Connectivity -> (none); Manufacturer 1 (none) -> TE Connectivity; Manufacturer Part Number 1 (none) -> 1-2199230-6; OldValue (none) -> Bus_M.2_1-2199230-6
- M3: OldValue (none) -> Mech_M2_2280_H2.5mm
- R13, R14, R15, R16, R17, R18, R19, R20, R29, R30, R31, R52: value R_0R_0402 -> ERJ2GE0R00X; MPN ERJ2GE0R00X -> (none); Manufacturer Panasonic -> (none); Manufacturer 1 (none) -> Panasonic; Manufacturer Part Number 1 (none) -> ERJ2GE0R00X; OldValue (none) -> R_0R_0402
- R143: value R_0R_22.4A_0603 -> PMR03EZPJ000; MPN PMR03EZPJ000 -> (none); Manufacturer ROHM Semiconductor -> (none); Manufacturer 1 (none) -> ROHM Semiconductor; Manufacturer Part Number 1 (none) -> PMR03EZPJ000; OldValue (none) -> R_0R_22.4A_0603
- R186, R187, R39: value R_200R_0402 -> CR0402-FX-2000GLF; MPN CR0402-FX-2000GLF -> (none); Manufacturer Bourns -> (none); Manufacturer 1 (none) -> Bourns; Manufacturer Part Number 1 (none) -> CR0402-FX-2000GLF; OldValue (none) -> R_200R_0402
- R21, R22: value R_4x0R_0201_array -> EXB-18VR000X; MPN EXB-18VR000X -> (none); Manufacturer Panasonic -> (none); Manufacturer 1 (none) -> Panasonic; Manufacturer Part Number 1 (none) -> EXB-18VR000X; OldValue (none) -> R_4x0R_0201_array
- R27, R28, R32, R37, R38: value R_47k_0402 -> CR0402-FX-4702GLF; MPN CR0402-FX-4702GLF -> (none); Manufacturer Bourns -> (none); Manufacturer 1 (none) -> Bourns; Manufacturer Part Number 1 (none) -> CR0402-FX-4702GLF; OldValue (none) -> R_47k_0402
- SP7, SP8: value Spacer_Drill3.7mm_H2.5mm_9774025151R -> 9774025151R; MPN 9774025151R -> (none); Manufacturer Würth Elektronik -> (none); Manufacturer 1 (none) -> Würth Elektronik; Manufacturer Part Number 1 (none) -> 9774025151R; OldValue (none) -> Spacer_Drill3.7mm_H2.5mm_9774025151R
- TP10, TP11, TP12, TP6, TP7, TP8, TP9: OldValue (none) -> TP_0.75mm_SMD
- U2, U3: value 74LVC2G07_SOT457 -> 74LVC2G07GV,125; MPN 74LVC2G07GV,125 -> (none); Manufacturer Nexperia -> (none); Manufacturer 1 (none) -> Nexperia; Manufacturer Part Number 1 (none) -> 74LVC2G07GV,125; OldValue (none) -> 74LVC2G07_SOT457
- Y1: value Oscillator_32.768kHz_ECS_2520MV -> ECS-327MVATX-2-CN-TR3; MPN ECS-327MVATX-2-CN-TR3 -> (none); Manufacturer ECS Inc. International -> (none); Manufacturer 1 (none) -> ECS Inc. International; Manufacturer Part Number 1 (none) -> ECS-327MVATX-2-CN-TR3; OldValue (none) -> Oscillator_32.768kHz_ECS_2520MV
