File: peripherals.kicad_sch (KiCad schematic)
At the start: 93 parts, among them J10 Molex_PicoBlade_1x4_0533980471, J11 Socket_Samtec_ERF8_2x40_ERF8-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, J14 JST_SH_1x4_SM04B-SRSS-TB-LF-SN, J9 Tag-Connect_TC2050-IDC-NL_2x5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, Q10 PJE138K, Q9 PJE138K, U30 TPD4E05U06QDQARQ1, U33 NTS0102_XSON, U34 PCAL6408A_VQFN, U35 AP22653_DFN

Commit message: Adding libs/3d-models back from commit 51986f3981aa7fd18fc8cc0c4764f958b589b418
Parts:
- C104, C111, C113, C130, C44, C48: value C_100n_0402 -> GRM155R61H104KE14D; MPN GRM155R61H104KE14D -> (none); Manufacturer Murata -> (none); Manufacturer 1 (none) -> Murata; Manufacturer Part Number 1 (none) -> GRM155R61H104KE14D; OldValue (none) -> C_100n_0402
- C105, C106, C107, C114, C115: value C_1u_0402 -> C1005X6S1A105K050BC; MPN C1005X6S1A105K050BC -> (none); Manufacturer TDK -> (none); Manufacturer 1 (none) -> TDK; Manufacturer Part Number 1 (none) -> C1005X6S1A105K050BC; OldValue (none) -> C_1u_0402
- C108, C109, C110, C112: value C_220n_0402 -> CC0402KRX5R6BB224; MPN CC0402KRX5R6BB224 -> (none); Manufacturer YAGEO -> (none); Manufacturer 1 (none) -> YAGEO; Manufacturer Part Number 1 (none) -> CC0402KRX5R6BB224; OldValue (none) -> C_220n_0402
- D16, D17, D19, D21, D22, D23, D39, D40, D41, D42, D43, D44, D45, D46, D47, D48, D49, D50, D56, D57, D58, D59: value TPD1E0B04_XDFN-2 -> TPD1E0B04DPYR; MPN TPD1E0B04DPYR -> (none); Manufacturer Texas Instruments -> (none); Manufacturer 1 (none) -> Texas Instruments; Manufacturer Part Number 1 (none) -> TPD1E0B04DPYR; OldValue (none) -> TPD1E0B04_XDFN-2
- D26, D27, D54: value LED_G_0603_LTST-C190GKT -> LTST-C190GKT; MPN LTST-C190GKT -> (none); Manufacturer Lite-On -> (none); Manufacturer 1 (none) -> Lite-On; Manufacturer Part Number 1 (none) -> LTST-C190GKT; OldValue (none) -> LED_G_0603_LTST-C190GKT
- D63: MPN RB521S30T1G -> (none); Manufacturer ON Semiconductor -> (none); Manufacturer 1 (none) -> ON Semiconductor; Manufacturer Part Number 1 (none) -> RB521S30T1G; OldValue (none) -> RB521S30T1G
- J10: value Molex_PicoBlade_1x4_0533980471 -> 0533980471; MPN 0533980471 -> (none); Manufacturer Molex -> (none); Manufacturer 1 (none) -> Molex; Manufacturer Part Number 1 (none) -> 0533980471; OldValue (none) -> Molex_PicoBlade_1x4_0533980471
- J11: value Socket_Samtec_ERF8_2x40_ERF8-040-05.0-L-DV-K-TR -> ERF8-040-05.0-L-DV-K-TR; MPN ERF8-040-05.0-L-DV-K-TR -> (none); Manufacturer Samtec -> (none); Manufacturer 1 (none) -> Samtec; Manufacturer Part Number 1 (none) -> ERF8-040-05.0-L-DV-K-TR; OldValue (none) -> Socket_Samtec_ERF8_2x40_ERF8-040-05.0-L-DV-K-TR
- J14: value JST_SH_1x4_SM04B-SRSS-TB-LF-SN -> SM04B-SRSS-TB(LF)(SN); MPN SM04B-SRSS-TB(LF)(SN) -> (none); Manufacturer JST Automotive Connectors -> (none); Manufacturer 1 (none) -> JST Automotive Connectors; Manufacturer Part Number 1 (none) -> SM04B-SRSS-TB(LF)(SN); OldValue (none) -> JST_SH_1x4_SM04B-SRSS-TB-LF-SN
- J9: value Tag-Connect_TC2050-IDC-NL_2x5_P1.27mm -> TC2050-IDC-NL; MPN TC2050-IDC-NL -> (none); Manufacturer Tag Connect -> (none); Manufacturer 1 (none) -> Tag Connect; Manufacturer Part Number 1 (none) -> TC2050-IDC-NL; OldValue (none) -> Tag-Connect_TC2050-IDC-NL_2x5_P1.27mm
- Q10, Q9: value PJE138K -> PJE138K_R1_00001; MPN PJE138K_R1_00001 -> (none); Manufacturer PANJIT -> (none); Manufacturer 1 (none) -> PANJIT; Manufacturer Part Number 1 (none) -> PJE138K_R1_00001; OldValue (none) -> PJE138K
- R100, R101, R102, R26, R53, R54, R63, R64: value R_4x330R_0402_array -> EXB-28V331JX; MPN EXB-28V331JX -> (none); Manufacturer Panasonic -> (none); Manufacturer 1 (none) -> Panasonic; Manufacturer Part Number 1 (none) -> EXB-28V331JX; OldValue (none) -> R_4x330R_0402_array
- R112: value R_4x100R_0201_array -> EXB-18V101JX; MPN EXB-18V101JX -> (none); Manufacturer Panasonic -> (none); Manufacturer 1 (none) -> Panasonic; Manufacturer Part Number 1 (none) -> EXB-18V101JX; OldValue (none) -> R_4x100R_0201_array
- R120, R121, R134, R141, R215, R216, R217, R218, R55, R62: value R_0R_0402 -> ERJ2GE0R00X; MPN ERJ2GE0R00X -> (none); Manufacturer Panasonic -> (none); Manufacturer 1 (none) -> Panasonic; Manufacturer Part Number 1 (none) -> ERJ2GE0R00X; OldValue (none) -> R_0R_0402
- R189, R219, R232, R242: value R_10k_0402 -> CR0402-FX-1002GLF; MPN CR0402-FX-1002GLF -> (none); Manufacturer Bourns -> (none); Manufacturer 1 (none) -> Bourns; Manufacturer Part Number 1 (none) -> CR0402-FX-1002GLF; OldValue (none) -> R_10k_0402
- R190: value R_15k_0402 -> CR0402-FX-1502GLF; MPN CR0402-FX-1502GLF -> (none); Manufacturer Bourns -> (none); Manufacturer 1 (none) -> Bourns; Manufacturer Part Number 1 (none) -> CR0402-FX-1502GLF; OldValue (none) -> R_15k_0402
- R191, R223, R231: value R_200R_0402 -> CR0402-FX-2000GLF; MPN CR0402-FX-2000GLF -> (none); Manufacturer Bourns -> (none); Manufacturer 1 (none) -> Bourns; Manufacturer Part Number 1 (none) -> CR0402-FX-2000GLF; OldValue (none) -> R_200R_0402
- R192, R222, R230: value R_100k_0402 -> CR0402-FX-1003GLF; MPN CR0402-FX-1003GLF -> (none); Manufacturer Bourns -> (none); Manufacturer 1 (none) -> Bourns; Manufacturer Part Number 1 (none) -> CR0402-FX-1003GLF; OldValue (none) -> R_100k_0402
- R195, R204, R25: value R_4x0R_0201_array -> EXB-18VR000X; MPN EXB-18VR000X -> (none); Manufacturer Panasonic -> (none); Manufacturer 1 (none) -> Panasonic; Manufacturer Part Number 1 (none) -> EXB-18VR000X; OldValue (none) -> R_4x0R_0201_array
- R233, R235, R248: value R_0R_22.4A_0603 -> PMR03EZPJ000; MPN PMR03EZPJ000 -> (none); Manufacturer ROHM Semiconductor -> (none); Manufacturer 1 (none) -> ROHM Semiconductor; Manufacturer Part Number 1 (none) -> PMR03EZPJ000; OldValue (none) -> R_0R_22.4A_0603
- R234, R247: value R_0R_0603 -> CR0603-J/-000ELF; MPN CR0603-J/-000ELF -> (none); Manufacturer Bourns -> (none); Manufacturer 1 (none) -> Bourns; Manufacturer Part Number 1 (none) -> CR0603-J/-000ELF; OldValue (none) -> R_0R_0603
- R335, R336: value R_470R_0402 -> CR0402-FX-4700GLF; MPN CR0402-FX-4700GLF -> (none); Manufacturer Bourns -> (none); Manufacturer 1 (none) -> Bourns; Manufacturer Part Number 1 (none) -> CR0402-FX-4700GLF; OldValue (none) -> R_470R_0402
- S2, S3: value SW_KMR211NGLFS_SMD -> KMR211NGLFS; MPN KMR211NGLFS -> (none); Manufacturer C&K -> (none); Manufacturer 1 (none) -> C&K; Manufacturer Part Number 1 (none) -> KMR211NGLFS; OldValue (none) -> SW_KMR211NGLFS_SMD
- U30: MPN TPD4E05U06QDQARQ1 -> (none); Manufacturer Texas Instruments -> (none); Manufacturer 1 (none) -> Texas Instruments; Manufacturer Part Number 1 (none) -> TPD4E05U06QDQARQ1; OldValue (none) -> TPD4E05U06QDQARQ1
- U33: value NTS0102_XSON -> NTS0102GT; MPN NTS0102GT -> (none); Manufacturer NXP -> (none); Manufacturer 1 (none) -> NXP; Manufacturer Part Number 1 (none) -> NTS0102GT; OldValue (none) -> NTS0102_XSON
- U34: value PCAL6408A_VQFN -> PCAL6408ABSHP; MPN PCAL6408ABSHP -> (none); Manufacturer NXP -> (none); Manufacturer 1 (none) -> NXP; Manufacturer Part Number 1 (none) -> PCAL6408ABSHP; OldValue (none) -> PCAL6408A_VQFN
- U35: value AP22653_DFN -> AP22653FDZ-7; MPN AP22653FDZ-7 -> (none); Manufacturer Diodes Incorporated -> (none); Manufacturer 1 (none) -> Diodes Incorporated; Manufacturer Part Number 1 (none) -> AP22653FDZ-7; OldValue (none) -> AP22653_DFN
