File: som.kicad_sch (KiCad schematic)
At the start: 29 parts, among them J15 Bus_DDR4_SODIMM_CUSTOM_Jetson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, M1 Jetson-Orin-NX-Nano, U4 NTS0102_XSON

Commit message: Adding libs/3d-models back from commit 51986f3981aa7fd18fc8cc0c4764f958b589b418
Parts:
- BT1: value Battery_Holder_MS621FE-FL11E -> MS621FE-FL11E; MPN MS621FE-FL11E -> (none); Manufacturer Seiko Instruments -> (none); Manufacturer 1 (none) -> Seiko Instruments; Manufacturer Part Number 1 (none) -> MS621FE-FL11E; OldValue (none) -> Battery_Holder_MS621FE-FL11E
- C1, C2: value C_Pol_100u_25V_KEMET-T521-D-107 -> T521D107M025ATE040; MPN T521D107M025ATE040 -> (none); Manufacturer KEMET -> (none); Manufacturer 1 (none) -> KEMET; Manufacturer Part Number 1 (none) -> T521D107M025ATE040; OldValue (none) -> C_Pol_100u_25V_KEMET-T521-D-107
- C40, C41: value C_100n_0402 -> GRM155R61H104KE14D; MPN GRM155R61H104KE14D -> (none); Manufacturer Murata -> (none); Manufacturer 1 (none) -> Murata; Manufacturer Part Number 1 (none) -> GRM155R61H104KE14D; OldValue (none) -> C_100n_0402
- D34: MPN RB521S30T1G -> (none); Manufacturer ON Semiconductor -> (none); Manufacturer 1 (none) -> ON Semiconductor; Manufacturer Part Number 1 (none) -> RB521S30T1G; OldValue (none) -> RB521S30T1G
- D55: value TPD1E0B04_XDFN-2 -> TPD1E0B04DPYR; MPN TPD1E0B04DPYR -> (none); Manufacturer Texas Instruments -> (none); Manufacturer 1 (none) -> Texas Instruments; Manufacturer Part Number 1 (none) -> TPD1E0B04DPYR; OldValue (none) -> TPD1E0B04_XDFN-2
- FB1: value FB_10Z_10A_WE-MPSB_1206 -> 74279221100; MPN 74279221100 -> (none); Manufacturer Würth Elektronik -> (none); Manufacturer 1 (none) -> Würth Elektronik; Manufacturer Part Number 1 (none) -> 74279221100; OldValue (none) -> FB_10Z_10A_WE-MPSB_1206
- H1, H2: value Spacer_Drill3.7mm_H6.5mm_9774065151R -> 9774065151R; MPN 9774065151R -> (none); Manufacturer Würth Elektronik -> (none); Manufacturer 1 (none) -> Würth Elektronik; Manufacturer Part Number 1 (none) -> 9774065151R; OldValue (none) -> Spacer_Drill3.7mm_H6.5mm_9774065151R
- J15: value Bus_DDR4_SODIMM_CUSTOM_Jetson-Orin-H9.2mm-socket -> 2309413-1; MPN 2309413-1 -> (none); Manufacturer TE Connectivity -> (none); Manufacturer 1 (none) -> TE Connectivity; Manufacturer Part Number 1 (none) -> 2309413-1; OldValue (none) -> Bus_DDR4_SODIMM_CUSTOM_Jetson-Orin-H9.2mm-socket
- M1: value Jetson-Orin-NX-Nano -> 900-13767-0000-000; MPN 900-13767-0000-000 -> (none); Manufacturer Nvidia -> (none); Manufacturer 1 (none) -> Nvidia; Manufacturer Part Number 1 (none) -> 900-13767-0000-000; OldValue (none) -> Jetson-Orin-NX-Nano
- R1, R11, R12, R2, R3, R4, R5: value R_0R_0402 -> ERJ2GE0R00X; MPN ERJ2GE0R00X -> (none); Manufacturer Panasonic -> (none); Manufacturer 1 (none) -> Panasonic; Manufacturer Part Number 1 (none) -> ERJ2GE0R00X; OldValue (none) -> R_0R_0402
- R294: value R_2k2_0402 -> CR0402-FX-2201GLF; MPN CR0402-FX-2201GLF -> (none); Manufacturer Bourns -> (none); Manufacturer 1 (none) -> Bourns; Manufacturer Part Number 1 (none) -> CR0402-FX-2201GLF; OldValue (none) -> R_2k2_0402
- R80: value R_4k7_0402 -> CR0402-FX-4701GLF; MPN CR0402-FX-4701GLF -> (none); Manufacturer Bourns -> (none); Manufacturer 1 (none) -> Bourns; Manufacturer Part Number 1 (none) -> CR0402-FX-4701GLF; OldValue (none) -> R_4k7_0402
- S1: value SW_KMR211NGLFS_SMD -> KMR211NGLFS; MPN KMR211NGLFS -> (none); Manufacturer C&K -> (none); Manufacturer 1 (none) -> C&K; Manufacturer Part Number 1 (none) -> KMR211NGLFS; OldValue (none) -> SW_KMR211NGLFS_SMD
- TP2, TP3, TP35, TP4, TP44, TP5: OldValue (none) -> TP_0.75mm_SMD
- U4: value NTS0102_XSON -> NTS0102GT; MPN NTS0102GT -> (none); Manufacturer NXP -> (none); Manufacturer 1 (none) -> NXP; Manufacturer Part Number 1 (none) -> NTS0102GT; OldValue (none) -> NTS0102_XSON
