File: supply.kicad_sch (KiCad schematic)
At the start: 118 parts, among them J12 Molex_Nano-Fit_1x2_SMD_105430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, Q11 PJE138K, Q13 BCM857BS-7-F, Q14 BCM857BS-7-F, Q15 SSM3J332R, Q16 SSM3J332R, Q18 SSM3J332R, Q5 PJE138K, Q6 SSM3J332R, Q7 PJE138K, Q8 PJE138K, SW1 SW_SPDT_PCM12SMTR, U1 SIC431AED-T1-GE3, U29 LM73100, U37 74LVC2G14_SOT457, U38 74LVC1G175_SOT457, U40 SIC431AED-T1-GE3, U41 NCP730BMT330_WSON, U42 TPS7A0518P_SOT23-5, U48 LM73100

Commit message: Adding libs/3d-models back from commit 51986f3981aa7fd18fc8cc0c4764f958b589b418
Parts:
- C102, C118, C119, C121, C124, C125, C157, C50, C6: value C_100n_0402 -> GRM155R61H104KE14D; MPN GRM155R61H104KE14D -> (none); Manufacturer Murata -> (none); Manufacturer 1 (none) -> Murata; Manufacturer Part Number 1 (none) -> GRM155R61H104KE14D; OldValue (none) -> C_100n_0402
- C103, C120, C126, C127, C128, C129, C153, C154: value C_22u_16V_0603 -> CL10A226MO7JZNC; MPN CL10A226MO7JZNC -> (none); Manufacturer Samsung Electro-Mechanics -> (none); Manufacturer 1 (none) -> Samsung Electro-Mechanics; Manufacturer Part Number 1 (none) -> CL10A226MO7JZNC; OldValue (none) -> C_22u_16V_0603
- C116, C117, C137, C83: value C_10u_0402 -> CC0402MRX5R5BB106; MPN CC0402MRX5R5BB106 -> (none); Manufacturer YAGEO -> (none); Manufacturer 1 (none) -> YAGEO; Manufacturer Part Number 1 (none) -> CC0402MRX5R5BB106; OldValue (none) -> C_10u_0402
- C122, C151, C152, C5: value C_22u_25V_0805 -> CL21A226MAYNNNE; MPN CL21A226MAYNNNE -> (none); Manufacturer Samsung Electro-Mechanics -> (none); Manufacturer 1 (none) -> Samsung Electro-Mechanics; Manufacturer Part Number 1 (none) -> CL21A226MAYNNNE; OldValue (none) -> C_22u_25V_0805
- C123, C142, C93: value C_1u_0402 -> C1005X6S1A105K050BC; MPN C1005X6S1A105K050BC -> (none); Manufacturer TDK -> (none); Manufacturer 1 (none) -> TDK; Manufacturer Part Number 1 (none) -> C1005X6S1A105K050BC; OldValue (none) -> C_1u_0402
- C134: value C_10u_25V_0603 -> C1608X5R1E106M080AC; MPN C1608X5R1E106M080AC -> (none); Manufacturer TDK -> (none); Manufacturer 1 (none) -> TDK; Manufacturer Part Number 1 (none) -> C1608X5R1E106M080AC; OldValue (none) -> C_10u_25V_0603
- C150: value C_1u_25V_0402 -> GRM155R61E105KE11J; MPN GRM155R61E105KE11J -> (none); Manufacturer Murata -> (none); Manufacturer 1 (none) -> Murata; Manufacturer Part Number 1 (none) -> GRM155R61E105KE11J; OldValue (none) -> C_1u_25V_0402
- C155, C156: value C_4u7_25V_0402 -> GRM155C61E475ME15J; MPN GRM155C61E475ME15J -> (none); Manufacturer Murata -> (none); Manufacturer 1 (none) -> Murata; Manufacturer Part Number 1 (none) -> GRM155C61E475ME15J; OldValue (none) -> C_4u7_25V_0402
- C160: value C_1n_0402 -> GRM1555C1H102JA01D; MPN GRM1555C1H102JA01D -> (none); Manufacturer Murata -> (none); Manufacturer 1 (none) -> Murata; Manufacturer Part Number 1 (none) -> GRM1555C1H102JA01D; OldValue (none) -> C_1n_0402
- C161: value C_1n_16V_X7R_0402 -> C0402C102J4RACTU; MPN C0402C102J4RACTU -> (none); Manufacturer KEMET -> (none); Manufacturer 1 (none) -> KEMET; Manufacturer Part Number 1 (none) -> C0402C102J4RACTU; OldValue (none) -> C_1n_16V_X7R_0402
- D28, D29: value DF2S30FS_SOD -> DF2S30FS; MPN DF2S30FS -> (none); Manufacturer Toshiba -> (none); Manufacturer 1 (none) -> Toshiba; Manufacturer Part Number 1 (none) -> DF2S30FS; OldValue (none) -> DF2S30FS_SOD
- D30, D31, D32, D33: MPN ESD9X5.0ST5G -> (none); Manufacturer ON Semiconductor -> (none); Manufacturer 1 (none) -> ON Semiconductor; Manufacturer Part Number 1 (none) -> ESD9X5.0ST5G; OldValue (none) -> ESD9X5.0ST5G
- D36, D37: MPN RB521S30T1G -> (none); Manufacturer ON Semiconductor -> (none); Manufacturer 1 (none) -> ON Semiconductor; Manufacturer Part Number 1 (none) -> RB521S30T1G; OldValue (none) -> RB521S30T1G
- D53: value LED_G_0603_LTST-C190GKT -> LTST-C190GKT; MPN LTST-C190GKT -> (none); Manufacturer Lite-On -> (none); Manufacturer 1 (none) -> Lite-On; Manufacturer Part Number 1 (none) -> LTST-C190GKT; OldValue (none) -> LED_G_0603_LTST-C190GKT
- D60, D61: value TPD1E0B04_XDFN-2 -> TPD1E0B04DPYR; MPN TPD1E0B04DPYR -> (none); Manufacturer Texas Instruments -> (none); Manufacturer 1 (none) -> Texas Instruments; Manufacturer Part Number 1 (none) -> TPD1E0B04DPYR; OldValue (none) -> TPD1E0B04_XDFN-2
- J12: value Molex_Nano-Fit_1x2_SMD_1054301202 -> 105430-1202; MPN 105430-1202 -> (none); Manufacturer Molex -> (none); Manufacturer 1 (none) -> Molex; Manufacturer Part Number 1 (none) -> 105430-1202; OldValue (none) -> Molex_Nano-Fit_1x2_SMD_1054301202
- L1: value L_560n_17.7A_Bourns-SRP5030CA -> SRP5030CA-R56M; MPN SRP5030CA-R56M -> (none); Manufacturer Bourns -> (none); Manufacturer 1 (none) -> Bourns; Manufacturer Part Number 1 (none) -> SRP5030CA-R56M; OldValue (none) -> L_560n_17.7A_Bourns-SRP5030CA
- L4: value L_1u_20A_Bourns-SRP6050CA -> SRP6050CA-1R0M; MPN SRP6050CA-1R0M -> (none); Manufacturer Bourns -> (none); Manufacturer 1 (none) -> Bourns; Manufacturer Part Number 1 (none) -> SRP6050CA-1R0M; OldValue (none) -> L_1u_20A_Bourns-SRP6050CA
- Q11, Q5, Q7, Q8: value PJE138K -> PJE138K_R1_00001; MPN PJE138K_R1_00001 -> (none); Manufacturer PANJIT -> (none); Manufacturer 1 (none) -> PANJIT; Manufacturer Part Number 1 (none) -> PJE138K_R1_00001; OldValue (none) -> PJE138K
- Q13, Q14: MPN BCM857BS-7-F -> (none); Manufacturer Diodes Incorporated -> (none); Manufacturer 1 (none) -> Diodes Incorporated; Manufacturer Part Number 1 (none) -> BCM857BS-7-F; OldValue (none) -> BCM857BS-7-F
- Q15, Q16, Q18, Q6: value SSM3J332R -> SSM3J332R,LF; MPN SSM3J332R,LF -> (none); Manufacturer Toshiba -> (none); Manufacturer 1 (none) -> Toshiba; Manufacturer Part Number 1 (none) -> SSM3J332R,LF; OldValue (none) -> SSM3J332R
- R159, R173, R176, R237, R239, R240: value R_499k_0402 -> CR0402-FX-4993GLF; MPN CR0402-FX-4993GLF -> (none); Manufacturer Bourns -> (none); Manufacturer 1 (none) -> Bourns; Manufacturer Part Number 1 (none) -> CR0402-FX-4993GLF; OldValue (none) -> R_499k_0402
- R164, R165: value R_4k7_0402 -> CR0402-FX-4701GLF; MPN CR0402-FX-4701GLF -> (none); Manufacturer Bourns -> (none); Manufacturer 1 (none) -> Bourns; Manufacturer Part Number 1 (none) -> CR0402-FX-4701GLF; OldValue (none) -> R_4k7_0402
- R169: value R_2k7_0402 -> CR0402-FX-2701GLF; MPN CR0402-FX-2701GLF -> (none); Manufacturer Bourns -> (none); Manufacturer 1 (none) -> Bourns; Manufacturer Part Number 1 (none) -> CR0402-FX-2701GLF; OldValue (none) -> R_2k7_0402
- R170: value R_73k2_0402 -> CR0402-FX-7322GLF; MPN CR0402-FX-7322GLF -> (none); Manufacturer Bourns -> (none); Manufacturer 1 (none) -> Bourns; Manufacturer Part Number 1 (none) -> CR0402-FX-7322GLF; OldValue (none) -> R_73k2_0402
- R172, R175, R178, R182, R252, R253: value R_0R_22.4A_0603 -> PMR03EZPJ000; MPN PMR03EZPJ000 -> (none); Manufacturer ROHM Semiconductor -> (none); Manufacturer 1 (none) -> ROHM Semiconductor; Manufacturer Part Number 1 (none) -> PMR03EZPJ000; OldValue (none) -> R_0R_22.4A_0603
- R177: value R_45k3_0402 -> CR0402-FX-4532GLF; MPN CR0402-FX-4532GLF -> (none); Manufacturer Bourns -> (none); Manufacturer 1 (none) -> Bourns; Manufacturer Part Number 1 (none) -> CR0402-FX-4532GLF; OldValue (none) -> R_45k3_0402
- R181, R188, R238, R250, R251, R254, R255, R259, R269, R275: value R_10k_0402 -> CR0402-FX-1002GLF; MPN CR0402-FX-1002GLF -> (none); Manufacturer Bourns -> (none); Manufacturer 1 (none) -> Bourns; Manufacturer Part Number 1 (none) -> CR0402-FX-1002GLF; OldValue (none) -> R_10k_0402
- R183, R260, R264, R268: value R_0R_0402 -> ERJ2GE0R00X; MPN ERJ2GE0R00X -> (none); Manufacturer Panasonic -> (none); Manufacturer 1 (none) -> Panasonic; Manufacturer Part Number 1 (none) -> ERJ2GE0R00X; OldValue (none) -> R_0R_0402
- R236: value R_200R_0402 -> CR0402-FX-2000GLF; MPN CR0402-FX-2000GLF -> (none); Manufacturer Bourns -> (none); Manufacturer 1 (none) -> Bourns; Manufacturer Part Number 1 (none) -> CR0402-FX-2000GLF; OldValue (none) -> R_200R_0402
- R249: value R_100k_0402 -> CR0402-FX-1003GLF; MPN CR0402-FX-1003GLF -> (none); Manufacturer Bourns -> (none); Manufacturer 1 (none) -> Bourns; Manufacturer Part Number 1 (none) -> CR0402-FX-1003GLF; OldValue (none) -> R_100k_0402
- R256: value R_1k_0402 -> CR0402-FX-1001GLF; MPN CR0402-FX-1001GLF -> (none); Manufacturer Bourns -> (none); Manufacturer 1 (none) -> Bourns; Manufacturer Part Number 1 (none) -> CR0402-FX-1001GLF; OldValue (none) -> R_1k_0402
- R257, R258, R261: value R_200k_0402 -> CR0402-FX-2003GLF; MPN CR0402-FX-2003GLF -> (none); Manufacturer Bourns -> (none); Manufacturer 1 (none) -> Bourns; Manufacturer Part Number 1 (none) -> CR0402-FX-2003GLF; OldValue (none) -> R_200k_0402
- R263: value R_20k_0402 -> CR0402-FX-2002GLF; MPN CR0402-FX-2002GLF -> (none); Manufacturer Bourns -> (none); Manufacturer 1 (none) -> Bourns; Manufacturer Part Number 1 (none) -> CR0402-FX-2002GLF; OldValue (none) -> R_20k_0402
- R272, R274: value R_470k_0402 -> CR0402-FX-4703GLF; MPN CR0402-FX-4703GLF -> (none); Manufacturer Bourns -> (none); Manufacturer 1 (none) -> Bourns; Manufacturer Part Number 1 (none) -> CR0402-FX-4703GLF; OldValue (none) -> R_470k_0402
- R273, R276: value R_0R_0603 -> CR0603-J/-000ELF; MPN CR0603-J/-000ELF -> (none); Manufacturer Bourns -> (none); Manufacturer 1 (none) -> Bourns; Manufacturer Part Number 1 (none) -> CR0603-J/-000ELF; OldValue (none) -> R_0R_0603
- S4, S5: value SW_KMR211NGLFS_SMD -> KMR211NGLFS; MPN KMR211NGLFS -> (none); Manufacturer C&K -> (none); Manufacturer 1 (none) -> C&K; Manufacturer Part Number 1 (none) -> KMR211NGLFS; OldValue (none) -> SW_KMR211NGLFS_SMD
- SW1: value SW_SPDT_PCM12SMTR -> PCM12SMTR; MPN PCM12SMTR -> (none); Manufacturer C&K -> (none); Manufacturer 1 (none) -> C&K; Manufacturer Part Number 1 (none) -> PCM12SMTR; OldValue (none) -> SW_SPDT_PCM12SMTR
- TP14, TP23, TP33, TP52, TP53, TP54, TP55: OldValue (none) -> TP_0.75mm_SMD
- U1, U40: MPN SIC431AED-T1-GE3 -> (none); Manufacturer Vishay -> (none); Manufacturer 1 (none) -> Vishay; Manufacturer Part Number 1 (none) -> SIC431AED-T1-GE3; OldValue (none) -> SIC431AED-T1-GE3
- U29, U48: value LM73100 -> LM73100RPWR; MPN LM73100RPWR -> (none); Manufacturer Texas Instruments -> (none); Manufacturer 1 (none) -> Texas Instruments; Manufacturer Part Number 1 (none) -> LM73100RPWR; OldValue (none) -> LM73100
- U37: value 74LVC2G14_SOT457 -> 74LVC2G14GV,125; MPN 74LVC2G14GV,125 -> (none); Manufacturer Nexperia -> (none); Manufacturer 1 (none) -> Nexperia; Manufacturer Part Number 1 (none) -> 74LVC2G14GV,125; OldValue (none) -> 74LVC2G14_SOT457
- U38: value 74LVC1G175_SOT457 -> 74LVC1G175GV,125; MPN 74LVC1G175GV,125 -> (none); Manufacturer Nexperia -> (none); Manufacturer 1 (none) -> Nexperia; Manufacturer Part Number 1 (none) -> 74LVC1G175GV,125; OldValue (none) -> 74LVC1G175_SOT457
- U41: value NCP730BMT330_WSON -> NCP730BMT330TBG; MPN NCP730BMT330TBG -> (none); Manufacturer ON Semiconductor -> (none); Manufacturer 1 (none) -> ON Semiconductor; Manufacturer Part Number 1 (none) -> NCP730BMT330TBG; OldValue (none) -> NCP730BMT330_WSON
- U42: value TPS7A0518P_SOT23-5 -> TPS7A0518PDBVT; MPN TPS7A0518PDBVT -> (none); Manufacturer Texas Instruments -> (none); Manufacturer 1 (none) -> Texas Instruments; Manufacturer Part Number 1 (none) -> TPS7A0518PDBVT; OldValue (none) -> TPS7A0518P_SOT23-5
