File: usb.kicad_sch (KiCad schematic)
At the start: 140 parts, among them J3 USB-C_GCT_USB4105-GF-A, J4 USB-C_WE_632723300011, Q20 PJE138K, Q21 PJE138K, U10 TUSB1046-DCIRNQ, U11 TPD4E05U06QDQARQ1, U12 AP22615A_TSOT26, U13 TPD4E05U06QDQARQ1, U14 TPD4E05U06QDQARQ1, U15 TPD4E05U06QDQARQ1, U16 TPD4E05U06QDQARQ1, U47 NTS0102_XSON, U5 FT230X_QFN, U6 TPS65988DHRSHR, U7 W25Q80DV_USON, U8 NCP730BMT330_WSON, U9 AP22615A_TSOT26

Commit message: Adding libs/3d-models back from commit 51986f3981aa7fd18fc8cc0c4764f958b589b418
Parts:
- C136, C148: value C_4u7_25V_0402 -> GRM155C61E475ME15J; MPN GRM155C61E475ME15J -> (none); Manufacturer Murata -> (none); Manufacturer 1 (none) -> Murata; Manufacturer Part Number 1 (none) -> GRM155C61E475ME15J; OldValue (none) -> C_4u7_25V_0402
- C140, C141, C143, C144, C158, C159, C26, C27, C29, C31, C33, C36, C37, C45, C53, C54, C55, C57, C58, C60, C61, C62, C63, C64, C65: value C_100n_0402 -> GRM155R61H104KE14D; MPN GRM155R61H104KE14D -> (none); Manufacturer Murata -> (none); Manufacturer 1 (none) -> Murata; Manufacturer Part Number 1 (none) -> GRM155R61H104KE14D; OldValue (none) -> C_100n_0402
- C145, C146: value C_47p_0402 -> C0402C470J5GACTU; MPN C0402C470J5GACTU -> (none); Manufacturer KEMET -> (none); Manufacturer 1 (none) -> KEMET; Manufacturer Part Number 1 (none) -> C0402C470J5GACTU; OldValue (none) -> C_47p_0402
- C147, C149: value C_1u_25V_0402 -> GRM155R61E105KE11J; MPN GRM155R61E105KE11J -> (none); Manufacturer Murata -> (none); Manufacturer 1 (none) -> Murata; Manufacturer Part Number 1 (none) -> GRM155R61E105KE11J; OldValue (none) -> C_1u_25V_0402
- C28, C30, C34, C35, C49, C56, C59: value C_10u_0402 -> CC0402MRX5R5BB106; MPN CC0402MRX5R5BB106 -> (none); Manufacturer YAGEO -> (none); Manufacturer 1 (none) -> YAGEO; Manufacturer Part Number 1 (none) -> CC0402MRX5R5BB106; OldValue (none) -> C_10u_0402
- C32: value C_10u_25V_0603 -> C1608X5R1E106M080AC; MPN C1608X5R1E106M080AC -> (none); Manufacturer TDK -> (none); Manufacturer 1 (none) -> TDK; Manufacturer Part Number 1 (none) -> C1608X5R1E106M080AC; OldValue (none) -> C_10u_25V_0603
- D2, D3, D4, D5, D8, D9: value LED_G_0603_LTST-C190GKT -> LTST-C190GKT; MPN LTST-C190GKT -> (none); Manufacturer Lite-On -> (none); Manufacturer 1 (none) -> Lite-On; Manufacturer Part Number 1 (none) -> LTST-C190GKT; OldValue (none) -> LED_G_0603_LTST-C190GKT
- D35: MPN RB521S30T1G -> (none); Manufacturer ON Semiconductor -> (none); Manufacturer 1 (none) -> ON Semiconductor; Manufacturer Part Number 1 (none) -> RB521S30T1G; OldValue (none) -> RB521S30T1G
- D6, D7: value DF2S30FS_SOD -> DF2S30FS; MPN DF2S30FS -> (none); Manufacturer Toshiba -> (none); Manufacturer 1 (none) -> Toshiba; Manufacturer Part Number 1 (none) -> DF2S30FS; OldValue (none) -> DF2S30FS_SOD
- J3: value USB-C_GCT_USB4105-GF-A -> USB4105-GF-A; MPN USB4105-GF-A -> (none); Manufacturer GCT -> (none); Manufacturer 1 (none) -> GCT; Manufacturer Part Number 1 (none) -> USB4105-GF-A; OldValue (none) -> USB-C_GCT_USB4105-GF-A
- J4: value USB-C_WE_632723300011 -> 632723300011; MPN 632723300011 -> (none); Manufacturer Würth Elektronik -> (none); Manufacturer 1 (none) -> Würth Elektronik; Manufacturer Part Number 1 (none) -> 632723300011; OldValue (none) -> USB-C_WE_632723300011
- Q20, Q21: value PJE138K -> PJE138K_R1_00001; MPN PJE138K_R1_00001 -> (none); Manufacturer PANJIT -> (none); Manufacturer 1 (none) -> PANJIT; Manufacturer Part Number 1 (none) -> PJE138K_R1_00001; OldValue (none) -> PJE138K
- R104, R78: value R_2k2_0402 -> CR0402-FX-2201GLF; MPN CR0402-FX-2201GLF -> (none); Manufacturer Bourns -> (none); Manufacturer 1 (none) -> Bourns; Manufacturer Part Number 1 (none) -> CR0402-FX-2201GLF; OldValue (none) -> R_2k2_0402
- R105, R106, R130, R246, R262, R81: value R_4k7_0402 -> CR0402-FX-4701GLF; MPN CR0402-FX-4701GLF -> (none); Manufacturer Bourns -> (none); Manufacturer 1 (none) -> Bourns; Manufacturer Part Number 1 (none) -> CR0402-FX-4701GLF; OldValue (none) -> R_4k7_0402
- R109, R110: value R_2M_0402 -> RC0402FR-072ML; MPN RC0402FR-072ML -> (none); Manufacturer YAGEO -> (none); Manufacturer 1 (none) -> YAGEO; Manufacturer Part Number 1 (none) -> RC0402FR-072ML; OldValue (none) -> R_2M_0402
- R111, R267, R85, R86, R87, R88, R89, R90, R91, R92, R93, R94, R95, R96, R97, R98: value R_1k_0402 -> CR0402-FX-1001GLF; MPN CR0402-FX-1001GLF -> (none); Manufacturer Bourns -> (none); Manufacturer 1 (none) -> Bourns; Manufacturer Part Number 1 (none) -> CR0402-FX-1001GLF; OldValue (none) -> R_1k_0402
- R117, R127: value R_27R_0402 -> CR0402-FX-27R0GLF; MPN CR0402-FX-27R0GLF -> (none); Manufacturer Bourns -> (none); Manufacturer 1 (none) -> Bourns; Manufacturer Part Number 1 (none) -> CR0402-FX-27R0GLF; OldValue (none) -> R_27R_0402
- R131, R42, R44, R46, R74, R77, R83, R99: value R_10k_0402 -> CR0402-FX-1002GLF; MPN CR0402-FX-1002GLF -> (none); Manufacturer Bourns -> (none); Manufacturer 1 (none) -> Bourns; Manufacturer Part Number 1 (none) -> CR0402-FX-1002GLF; OldValue (none) -> R_10k_0402
- R144, R158, R244, R41, R56, R57, R58, R59, R65, R70, R71, R75, R76, R79, R82, R84: value R_0R_0402 -> ERJ2GE0R00X; MPN ERJ2GE0R00X -> (none); Manufacturer Panasonic -> (none); Manufacturer 1 (none) -> Panasonic; Manufacturer Part Number 1 (none) -> ERJ2GE0R00X; OldValue (none) -> R_0R_0402
- R205, R207, R270, R43, R45: value R_100k_0402 -> CR0402-FX-1003GLF; MPN CR0402-FX-1003GLF -> (none); Manufacturer Bourns -> (none); Manufacturer 1 (none) -> Bourns; Manufacturer Part Number 1 (none) -> CR0402-FX-1003GLF; OldValue (none) -> R_100k_0402
- R271: value R_10M_0402 -> CR0402-FX-1005GLF; MPN CR0402-FX-1005GLF -> (none); Manufacturer Bourns -> (none); Manufacturer 1 (none) -> Bourns; Manufacturer Part Number 1 (none) -> CR0402-FX-1005GLF; OldValue (none) -> R_10M_0402
- R33: value R_4x0R_0201_array -> EXB-18VR000X; MPN EXB-18VR000X -> (none); Manufacturer Panasonic -> (none); Manufacturer 1 (none) -> Panasonic; Manufacturer Part Number 1 (none) -> EXB-18VR000X; OldValue (none) -> R_4x0R_0201_array
- R68, R69, R72, R73: value R_200R_0402 -> CR0402-FX-2000GLF; MPN CR0402-FX-2000GLF -> (none); Manufacturer Bourns -> (none); Manufacturer 1 (none) -> Bourns; Manufacturer Part Number 1 (none) -> CR0402-FX-2000GLF; OldValue (none) -> R_200R_0402
- TP1, TP13, TP17, TP18, TP19, TP20, TP24, TP25, TP26, TP27, TP28, TP30: OldValue (none) -> TP_0.75mm_SMD
- U10: value TUSB1046-DCIRNQ -> TUSB1046-DCIRNQT; MPN TUSB1046-DCIRNQT -> (none); Manufacturer Texas Instruments -> (none); Manufacturer 1 (none) -> Texas Instruments; Manufacturer Part Number 1 (none) -> TUSB1046-DCIRNQT; OldValue (none) -> TUSB1046-DCIRNQ
- U11, U13, U14, U15, U16: MPN TPD4E05U06QDQARQ1 -> (none); Manufacturer Texas Instruments -> (none); Manufacturer 1 (none) -> Texas Instruments; Manufacturer Part Number 1 (none) -> TPD4E05U06QDQARQ1; OldValue (none) -> TPD4E05U06QDQARQ1
- U12, U9: value AP22615A_TSOT26 -> AP22615AWU-7; MPN AP22615AWU-7 -> (none); Manufacturer Diodes Incorporated -> (none); Manufacturer 1 (none) -> Diodes Incorporated; Manufacturer Part Number 1 (none) -> AP22615AWU-7; OldValue (none) -> AP22615A_TSOT26
- U47: value NTS0102_XSON -> NTS0102GT; MPN NTS0102GT -> (none); Manufacturer NXP -> (none); Manufacturer 1 (none) -> NXP; Manufacturer Part Number 1 (none) -> NTS0102GT; OldValue (none) -> NTS0102_XSON
- U5: value FT230X_QFN -> FT230XQ-R; MPN FT230XQ-R -> (none); Manufacturer FTDI Chip -> (none); Manufacturer 1 (none) -> FTDI Chip; Manufacturer Part Number 1 (none) -> FT230XQ-R; OldValue (none) -> FT230X_QFN
- U6: MPN TPS65988DHRSHR -> (none); Manufacturer Texas Instruments -> (none); Manufacturer 1 (none) -> Texas Instruments; Manufacturer Part Number 1 (none) -> TPS65988DHRSHR; OldValue (none) -> TPS65988DHRSHR
- U7: value W25Q80DV_USON -> W25Q80DVUXIE TR; MPN W25Q80DVUXIE TR -> (none); Manufacturer Winbond -> (none); Manufacturer 1 (none) -> Winbond; Manufacturer Part Number 1 (none) -> W25Q80DVUXIE TR; OldValue (none) -> W25Q80DV_USON
- U8: value NCP730BMT330_WSON -> NCP730BMT330TBG; MPN NCP730BMT330TBG -> (none); Manufacturer ON Semiconductor -> (none); Manufacturer 1 (none) -> ON Semiconductor; Manufacturer Part Number 1 (none) -> NCP730BMT330TBG; OldValue (none) -> NCP730BMT330_WSON
