File: usb3.kicad_sch (KiCad schematic)
At the start: 51 parts, among them J5 USB-C_WE_632723300011, Q19 PJE138K, Q4 PJE138K, U17 HD3SS3220RNH, U18 AP22615A_TSOT26, U19 TPD4E05U06QDQARQ1, U20 TPD4E05U06QDQARQ1, U21 TPD4E05U06QDQARQ1

Commit message: Adding libs/3d-models back from commit 51986f3981aa7fd18fc8cc0c4764f958b589b418
Parts:
- C66, C74: value C_10u_0603 -> GRM188R61A106KE69D; MPN GRM188R61A106KE69D -> (none); Manufacturer Murata -> (none); Manufacturer 1 (none) -> Murata; Manufacturer Part Number 1 (none) -> GRM188R61A106KE69D; OldValue (none) -> C_10u_0603
- C67, C68, C69, C70, C71, C72, C73, C75: value C_100n_0402 -> GRM155R61H104KE14D; MPN GRM155R61H104KE14D -> (none); Manufacturer Murata -> (none); Manufacturer 1 (none) -> Murata; Manufacturer Part Number 1 (none) -> GRM155R61H104KE14D; OldValue (none) -> C_100n_0402
- D10: MPN ESD9X5.0ST5G -> (none); Manufacturer ON Semiconductor -> (none); Manufacturer 1 (none) -> ON Semiconductor; Manufacturer Part Number 1 (none) -> ESD9X5.0ST5G; OldValue (none) -> ESD9X5.0ST5G
- D11: value LED_G_0603_LTST-C190GKT -> LTST-C190GKT; MPN LTST-C190GKT -> (none); Manufacturer Lite-On -> (none); Manufacturer 1 (none) -> Lite-On; Manufacturer Part Number 1 (none) -> LTST-C190GKT; OldValue (none) -> LED_G_0603_LTST-C190GKT
- J5: value USB-C_WE_632723300011 -> 632723300011; MPN 632723300011 -> (none); Manufacturer Würth Elektronik -> (none); Manufacturer 1 (none) -> Würth Elektronik; Manufacturer Part Number 1 (none) -> 632723300011; OldValue (none) -> USB-C_WE_632723300011
- Q19, Q4: value PJE138K -> PJE138K_R1_00001; MPN PJE138K_R1_00001 -> (none); Manufacturer PANJIT -> (none); Manufacturer 1 (none) -> PANJIT; Manufacturer Part Number 1 (none) -> PJE138K_R1_00001; OldValue (none) -> PJE138K
- R113, R114, R118, R119, R124, R125, R200, R201, R202, R203, R23, R245: value R_0R_0402 -> ERJ2GE0R00X; MPN ERJ2GE0R00X -> (none); Manufacturer Panasonic -> (none); Manufacturer 1 (none) -> Panasonic; Manufacturer Part Number 1 (none) -> ERJ2GE0R00X; OldValue (none) -> R_0R_0402
- R115, R116, R135, R136, R137, R138, R24, R60: value R_10k_0402 -> CR0402-FX-1002GLF; MPN CR0402-FX-1002GLF -> (none); Manufacturer Bourns -> (none); Manufacturer 1 (none) -> Bourns; Manufacturer Part Number 1 (none) -> CR0402-FX-1002GLF; OldValue (none) -> R_10k_0402
- R126, R265, R266, R61: value R_200k_0402 -> CR0402-FX-2003GLF; MPN CR0402-FX-2003GLF -> (none); Manufacturer Bourns -> (none); Manufacturer 1 (none) -> Bourns; Manufacturer Part Number 1 (none) -> CR0402-FX-2003GLF; OldValue (none) -> R_200k_0402
- R128: value R_887k_0402 -> ERJ-2RKF8873X; MPN ERJ-2RKF8873X -> (none); Manufacturer Panasonic -> (none); Manufacturer 1 (none) -> Panasonic; Manufacturer Part Number 1 (none) -> ERJ-2RKF8873X; OldValue (none) -> R_887k_0402
- R139: value R_2k2_0402 -> CR0402-FX-2201GLF; MPN CR0402-FX-2201GLF -> (none); Manufacturer Bourns -> (none); Manufacturer 1 (none) -> Bourns; Manufacturer Part Number 1 (none) -> CR0402-FX-2201GLF; OldValue (none) -> R_2k2_0402
- R140: value R_470R_0402 -> CR0402-FX-4700GLF; MPN CR0402-FX-4700GLF -> (none); Manufacturer Bourns -> (none); Manufacturer 1 (none) -> Bourns; Manufacturer Part Number 1 (none) -> CR0402-FX-4700GLF; OldValue (none) -> R_470R_0402
- R184: value R_1k_0402 -> CR0402-FX-1001GLF; MPN CR0402-FX-1001GLF -> (none); Manufacturer Bourns -> (none); Manufacturer 1 (none) -> Bourns; Manufacturer Part Number 1 (none) -> CR0402-FX-1001GLF; OldValue (none) -> R_1k_0402
- TP29, TP31, TP32: OldValue (none) -> TP_0.75mm_SMD
- U17: value HD3SS3220RNH -> HD3SS3220RNHT; MPN HD3SS3220RNHT -> (none); Manufacturer Texas Instruments -> (none); Manufacturer 1 (none) -> Texas Instruments; Manufacturer Part Number 1 (none) -> HD3SS3220RNHT; OldValue (none) -> HD3SS3220RNH
- U18: value AP22615A_TSOT26 -> AP22615AWU-7; MPN AP22615AWU-7 -> (none); Manufacturer Diodes Incorporated -> (none); Manufacturer 1 (none) -> Diodes Incorporated; Manufacturer Part Number 1 (none) -> AP22615AWU-7; OldValue (none) -> AP22615A_TSOT26
- U19, U20, U21: MPN TPD4E05U06QDQARQ1 -> (none); Manufacturer Texas Instruments -> (none); Manufacturer 1 (none) -> Texas Instruments; Manufacturer Part Number 1 (none) -> TPD4E05U06QDQARQ1; OldValue (none) -> TPD4E05U06QDQARQ1
